File: hardware/pcb/glove-v3.1/glove-v3.1.kicad_pcb (KiCad board)
At the start: 4 copper layers, 79 x 35 mm, 42 parts, among them U1 XIAO-ESP32C3, U2 CD74HC4067M96, U3 2.5x3mm-BUTTON

Commit message: updating v3.1
Parts:
- C16: value C-0402-0.1uF -> C-0402-0.1uF-16V
- moved U3 0.56 mm to (151.7, 53.7)
Routing:
- net /S2: track 2.69 -> 13.6 mm
- net /HALL_0: track 39.4 -> 49.8 mm
- net /HALL_1: track 40.6 -> 50.2 mm
- net /HALL_2: track 42.3 -> 51.2 mm
- net /HALL_3: track 44.1 -> 52.2 mm
- net /HALL_4: track 46.0 -> 53.5 mm
- net /S3: track 1.83 -> 9.01 mm
- net /HALL_5: track 42.6 -> 49.4 mm
- net /MUX_OUT: track 26.6 -> 33.2 mm
- net /HALL_6: track 37.9 -> 43.9 mm
- net /HALL_7: track 33.8 -> 39.1 mm
- net /S0: track 18.4 -> 23.0 mm
- net /S1: track 12.8 -> 13.9 mm
- net Net-(U1-PA7_A8_D8_SCK): track 12.6 -> 12.1 mm
