File: hardware/pcb/glove-v3.1/glove-v3.1.kicad_sch (KiCad schematic)
At the start: 36 parts, among them U1 XIAO-ESP32C3, U2 CD74HC4067M96, U3 2.5x3mm-BUTTON

Commit message: updating v3.1
Parts:
- removed C16: C-0402-0.1uF, 0_easyeda2kicad:C0402, symbol 0_easyeda2kicad:C-0402-0.1uF
- added C16: C-0402-0.1uF-16V, 0_easyeda2kicad:C0402, symbol 0_easyeda2kicad:C-0402-0.1uF-16V
Connections:
- net +3V3: now also C16.1
- net GND: now also C16.2
